File: EZ48.kicad_sch (KiCad schematic)
At the start: 29 parts, among them U1 74LS139, U2 74LS08, U3 74LS32, U4 74LS02, U5 74LS138

Commit message: Add files via upload
Parts:
- removed C10, C11, C12, C13, C14, C15, C16, C17, C18, C19, C2, C20, C21, C22, C23, C3, C4, C5, C6, C7, C8, C9: 47uF, Capacitor_THT:C_Disc_D7.5mm_W4.4mm_P5.00mm, symbol Device:C
- removed unit 4 of U2
- removed unit 3 of U2
- removed unit 4 of U3
- removed unit 3 of U3
- removed unit 2 of U3
- removed unit 3 of U4
- removed unit 4 of U4
- removed unit 2 of U4
- added C50: 0.1uF, Capacitor_THT:C_Disc_D7.5mm_W4.4mm_P5.00mm, symbol Device:C
- added C51: 10 uF, Capacitor_THT:C_Disc_D9.0mm_W5.0mm_P7.50mm, symbol Device:C
- added R2: 1M Ohm, Resistor_THT:R_Axial_DIN0411_L9.9mm_D3.6mm_P7.62mm_Vertical, symbol Device:R
- added R3: 47K Ohm, Resistor_THT:R_Axial_DIN0411_L9.9mm_D3.6mm_P7.62mm_Vertical, symbol Device:R
- added R4: 1K Ohm, Resistor_THT:R_Axial_DIN0411_L9.9mm_D3.6mm_P7.62mm_Vertical, symbol Device:R
- added U6: NE556, Package_DIP:DIP-14_W7.62mm_LongPads, symbol Timer:NE556
- added U7: 74LS02, Package_DIP:DIP-14_W7.62mm_LongPads, symbol 74xx:74LS02
Connections:
- net +5VDC: now also U2.14 (VCC), U3.14 (VCC), U4.14 (VCC), C50.2, R2.1, R3.2, R4.1, U6.10 (R), U6.14 (VCC)
- net GND: now also U2.7 (GND), U3.7 (GND), U4.7 (GND), C50.1, C51.2, U6.7 (GND)
- new net: C51.1, R3.1, U6.12 (THR), U6.13 (DIS)
- new net: R2.2, U6.8 (TR)
- new net: U6.9 (Q), U7.5, U7.6
- new net RESET: R4.2, U7.4
- no-connect marks 0 -> 1
Other:
- added sheet Bypass Caps (caps.kicad_sch)
- added sheet Unused Parts (unused.kicad_sch)
- note added: "ADDRESS DECODING LOGIC"
- note added: "RESET LOGIC"
- moved on the sheet: U1C, U2E, U3E, U4E
