File: EZ48.kicad_pcb (KiCad board)
At the start: 2 copper layers, 63 parts, among them IC1 2732, IC2 2732, IC3 2732, U1 74LS139, U2 74LS06, U5 74LS138, U6 NE556, U8 74LS06

Commit message: Add files via upload
Parts:
- added C1: 47uF, Capacitor_THT:C_Disc_D9.0mm_W5.0mm_P7.50mm, F.Cu at (160.9, 52.5)
- added C50: 0.1uF, Capacitor_THT:C_Disc_D7.5mm_W4.4mm_P5.00mm, F.Cu at (136.0, 88.5)
- added C51: 10 uF, Capacitor_THT:C_Disc_D9.0mm_W5.0mm_P7.50mm, F.Cu at (135.8, 82.2)
- added R1: 47Ohm, Resistor_THT:R_Axial_DIN0411_L9.9mm_D3.6mm_P7.62mm_Vertical, F.Cu at (161.8, 46.7)
- added R2: 1M Ohm, Resistor_THT:R_Axial_DIN0411_L9.9mm_D3.6mm_P7.62mm_Vertical, F.Cu at (136.6, 66.1)
- added R3: 47K Ohm, Resistor_THT:R_Axial_DIN0411_L9.9mm_D3.6mm_P7.62mm_Vertical, F.Cu at (136.6, 71.2)
- added R4: 1K Ohm, Resistor_THT:R_Axial_DIN0411_L9.9mm_D3.6mm_P7.62mm_Vertical, F.Cu at (136.6, 76.4)
- added U2: 74LS06, Package_DIP:DIP-14_W7.62mm_LongPads, F.Cu at (135.9, 46.2)
- added U3: NE556, Package_DIP:DIP-14_W7.62mm_LongPads, F.Cu at (147.6, 46.2)
- added U4: 6502, Package_DIP:DIP-40_W15.24mm, F.Cu at (117.2, 46.2)
- moved C42 70.1 mm to (120.0, 37.5)
- moved R4 11.5 mm to (54.5, 187.5)
Connections:
- net EXP0 renamed ~{EXP0}
- net EXP1 renamed ~{EXP1}
- net EXP2 renamed ~{EXP2}
- net EXP3 renamed ~{EXP3}
- net EXP4 renamed ~{EXP4}
- net PIASEL renamed ~{PIASEL}
- net RAMBANK1 renamed ~{RAMBANK1}
- net RAMBANK2 renamed ~{RAMBANK2}
- net RAMBANK3 renamed ~{RAMBANK3}
- net ROMBANK1 renamed ~{ROMBANK1}
- net ROMBANK2 renamed ~{ROMBANK2}
- net ROMBANK3 renamed ~{ROMBANK3}
- net SPEECHSEL renamed ~{SPEECHSEL}
- net VDPSEL renamed ~{VDPSEL}
