File: caps.kicad_sch (KiCad schematic)
At the start: 48 parts

Commit message: Add files via upload
Changed lines of the file:
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@@
 	)
 	(global_label "GND"
-		(shape input)
+		(shape passive)
 		(at 275.59 22.86 0)
 		(fields_autoplaced yes)
@@
 		)
 		(property "Intersheetrefs" "${INTERSHEET_REFS}"
-			(at 282.4457 22.86 0)
+			(at 281.3344 22.86 0)
 			(effects
 				(font
@@
 	)
 	(global_label "GND"
-		(shape input)
+		(shape passive)
 		(at 275.59 35.56 0)
 		(fields_autoplaced yes)
@@
 		)
 		(property "Intersheetrefs" "${INTERSHEET_REFS}"
-			(at 282.4457 35.56 0)
+			(at 281.3344 35.56 0)
 			(effects
 				(font
