File: video.kicad_sch (KiCad schematic)
At the start: 12 parts, among them J1 Conn_Coaxial, J2 Conn_Coaxial, Q1 2N4401, U6 TMS9918A, Y1 10.738635MHz

Commit message: Add files via upload
Connections:
- net AD0: now reaches U6.10 (AD0)
- net AD0: now also S1.14 (Q)
- net VRAM~{WE}: now reaches U6.11 (R/~{W})
- net VRAM~{WE}: now also S1.3 (~{WE})
- net ~{CSW}: now reaches U6.14 (~{CSW})
- net ~{CSR}: now reaches U6.15 (~{CSR})
- net ~{NMI}: now reaches U6.16 (~{INT})
- net AD7: now reaches U6.3 (AD7)
- net ~{RESET}: now reaches U6.34 (~{RESET}/SYNC)
- net AD6: now reaches U6.4 (AD6)
- net AD5: now reaches U6.5 (AD5)
- net AD4: now reaches U6.6 (AD4)
- net AD3: now reaches U6.7 (AD3)
- net AD2: now reaches U6.8 (AD2)
- net AD1: now reaches U6.9 (AD1)
- net ~{CAS} renamed VRAM~{CAS}
- net ~{RAS} renamed VRAM~{RAS}
Other:
- note added: "VIDEO DISPLAY PROCESSOR"
- moved on the sheet: C52, C53, C54, J1, J2, L1, Q1, R5, R7, S1, U6, Y1

Commit message: Add files via upload
Parts:
- removed C52, C53: 16pf, Capacitor_THT:C_Disc_D3.0mm_W1.6mm_P2.50mm, symbol Device:C
- removed C54: 0.1uf, Capacitor_THT:C_Disc_D3.0mm_W1.6mm_P2.50mm, symbol Device:C
- removed J1, J2: Conn_Coaxial, w_conn_av:KLPX-0848A, symbol Connector:Conn_Coaxial
- removed L1: Ferrite_Bead, Resistor_THT:R_Axial_DIN0207_L6.3mm_D2.5mm_P7.62mm_Horizontal, symbol Device:Ferrite_Bead
- removed Q1: 2N4401, Package_TO_SOT_THT:TO-92, symbol Device:Q_NPN_EBC
- removed R5: 75, Resistor_THT:R_Axial_DIN0207_L6.3mm_D2.5mm_P7.62mm_Horizontal, symbol Device:R
- removed R7: 470, Resistor_THT:R_Axial_DIN0207_L6.3mm_D2.5mm_P7.62mm_Horizontal, symbol Device:R
- removed Y1: 10.738635MHz, Crystal:Crystal_HC49-4H_Vertical, symbol Device:Crystal
Connections:
- net AD0: now also S1.2 (D); no longer S1.14 (Q)
- net XTAL1: now reaches U6.39 (XTAL1)
- net COMVID: now reaches U6.36 (COMVID)
- net VIDIN: now reaches U6.35 (EXTVDP)
- net XTAL2: now reaches U6.40 (XTAL2)
