File: unused.kicad_sch (KiCad schematic)
At the start: 4 parts, among them U2 74LS08, U3 74LS32, U4 74LS02, U6 NE556

Commit message: Add files via upload
Parts:
- removed U2: 74LS08, symbol 74xx:74LS08
- removed U3: 74LS32, Package_DIP:DIP-14_W7.62mm_LongPads, symbol 74xx:74LS32
- removed U4: 74LS02, Package_DIP:DIP-14_W7.62mm_LongPads, symbol 74xx:74LS02
- added C1: 47uF, Capacitor_THT:C_Disc_D9.0mm_W5.0mm_P7.50mm, symbol Device:C
- added R1: 47Ohm, Resistor_THT:R_Axial_DIN0411_L9.9mm_D3.6mm_P7.62mm_Vertical, symbol Device:R
- added U1: 74LS139, symbol 74xx:74LS139
- added U2: 74LS06, Package_DIP:DIP-14_W7.62mm_LongPads, symbol 74xx:74LS06
- renumbered U6 to U3
Connections:
- net +5VDC: now also U1.16 (VCC), U2.14 (VCC)
- net GND: now also C1.1, R1.2, U1.8 (GND), U2.7 (GND)
- new net: C1.2, R1.1
- no-connect marks 30 -> 16

Commit message: Add files via upload
Changed lines of the file:
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@@
 	)
 	(global_label "GND"
-		(shape input)
+		(shape passive)
 		(at 29.21 137.16 0)
 		(fields_autoplaced yes)
@@
 		)
 		(property "Intersheetrefs" "${INTERSHEET_REFS}"
-			(at 36.0657 137.16 0)
+			(at 34.9544 137.16 0)
 			(effects
 				(font
@@
 	)
 	(global_label "GND"
-		(shape input)
+		(shape passive)
 		(at 237.49 53.34 270)
 		(fields_autoplaced yes)
@@
 		)
 		(property "Intersheetrefs" "${INTERSHEET_REFS}"
-			(at 237.49 60.1957 90)
+			(at 237.49 59.0844 90)
 			(effects
 				(font
@@
 	)
 	(global_label "GND"
-		(shape input)
+		(shape passive)
 		(at 257.81 54.61 270)
 		(fields_autoplaced yes)
@@
 		)
 		(property "Intersheetrefs" "${INTERSHEET_REFS}"
-			(at 257.81 61.4657 90)
+			(at 257.81 60.3544 90)
 			(effects
 				(font
@@
 	)
 	(global_label "GND"
-		(shape input)
+		(shape passive)
 		(at 275.59 35.56 90)
 		(fields_autoplaced yes)
@@
 		)
 		(property "Intersheetrefs" "${INTERSHEET_REFS}"
-			(at 275.59 28.7043 90)
+			(at 275.59 29.8156 90)
 			(effects
 				(font

Commit message: Add files via upload
Parts:
- added U4: 6502, Package_DIP:DIP-40_W15.24mm_LongPads, symbol 65xx:6502
Connections:
- net +5VDC: now also U4.8 (VCC)
- net GND: now also U4.1 (VSS), U4.21 (VSS)
- new net A0: U4.9 (A0)
- new net A1: U4.10 (A1)
- new net A10: U4.19 (A10)
- new net A11: U4.20 (A11)
- new net A12: U4.22 (A12)
- new net A13: U4.23 (A13)
- new net A14: U4.24 (A14)
- new net A15: U4.25 (A15)
- new net A2: U4.11 (A2)
- new net A3: U4.12 (A3)
- new net A4: U4.13 (A4)
- new net A5: U4.14 (A5)
- new net A6: U4.15 (A6)
- new net A7: U4.16 (A7)
- new net A8: U4.17 (A8)
- new net A9: U4.18 (A9)
- new net D0: U4.33 (D0)
- new net D1: U4.32 (D1)
- new net D2: U4.31 (D2)
- new net D3: U4.30 (D3)
- new net D4: U4.29 (D4)
- new net D5: U4.28 (D5)
- new net D6: U4.27 (D6)
- new net D7: U4.26 (D7)
- new net R/~{W}: U4.34 (R/~{W})
- new net ~{NMI}: U4.6 (~{NMI})
- new net ~{RESET}: U4.40 (~{RES})

Commit message: Add files via upload
Parts:
- added R10, R7, R8, R9: 2200 Ohm, symbol Device:R
- added Y2: 10.738635MHz, Crystal:Crystal_HC49-4H_Vertical, symbol Device:Crystal
Connections:
- net +5VDC: now also R10.1, R7.1, R8.2, R9.1
- net ~{NMI}: now also R8.1
- net at U4.2 (RDY): now also R10.2
- net at U4.38 (~{SO}): now also R9.2
- net ~{IRQ}: now reaches U4.4 (~{IRQ})
- net ~{IRQ}: now also R7.2
- no-connect marks 16 -> 15
Other:
- moved on the sheet: U2B
